File: TranceiverV1/TranceiverV1.kicad_pcb (KiCad board)
At the start: 2 copper layers, 94.6 x 45.6 mm, 19 parts, among them J1 Conn_01x03_Socket, J3 Battery, U1 NRF24L01_, U3 102010388, U4 LD1086DTTR

Commit message: udpated spacing
Parts:
- moved C4 2.40 mm to (138.6, 112.5)
- moved R2 1.21 mm to (144.9, 134.0)
- moved R3 1.17 mm to (144.0, 112.4)
- moved R4 1.00 mm to (154.6, 134.0)
Routing:
- net /LED_ON1: track 19.1 -> 17.7 mm
- net /5V_IN: track 24.4 -> 25.6 mm
- net Net-(D2-A): track 4.32 -> 5.46 mm
- net Net-(D1-A): track 4.28 -> 5.36 mm
- net /LED_ON2: track 17.2 -> 16.2 mm
- net Net-(D3-A): track 4.80 -> 5.44 mm
Changed lines of the file:
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@@
 	(footprint "Capacitor_THT:C_Axial_L3.8mm_D2.6mm_P7.50mm_Horizontal"
 		(layer "F.Cu")
-		(at 140.8 111.575 -90)
+		(at 138.601627 112.525686 -90)
 		(descr "C, Axial series, Axial, Horizontal, pin pitch=7.5mm, length*diameter=3.8*2.6mm^2, http://www.vishay.com/docs/45231/arseries.pdf")
 		(tags "C Axial series Axial Horizontal pin pitch 7.5mm  length 3.8mm diameter 2.6mm")
@@
 	(footprint "Resistor_THT:R_Axial_DIN0204_L3.6mm_D1.6mm_P2.54mm_Vertical"
 		(layer "F.Cu")
-		(at 154.62 135 180)
+		(at 154.6 134 180)
 		(descr "Resistor, Axial_DIN0204 series, Axial, Vertical, pin pitch=2.54mm, 0.167W, length*diameter=3.6*1.6mm^2, http://cdn-reichelt.de/documents/datenblatt/B400/1_4W%23YAG.pdf")
 		(tags "Resistor Axial_DIN0204 series Axial Vertical pin pitch 2.54mm 0.167W length 3.6mm diameter 1.6mm")
@@
 	(footprint "Resistor_THT:R_Axial_DIN0204_L3.6mm_D1.6mm_P2.54mm_Vertical"
 		(layer "F.Cu")
-		(at 144.83 111.575 -90)
+		(at 144 112.4 -90)
 		(descr "Resistor, Axial_DIN0204 series, Axial, Vertical, pin pitch=2.54mm, 0.167W, length*diameter=3.6*1.6mm^2, http://cdn-reichelt.de/documents/datenblatt/B400/1_4W%23YAG.pdf")
 		(tags "Resistor Axial_DIN0204 series Axial Vertical pin pitch 2.54mm 0.167W length 3.6mm diameter 1.6mm")
@@
 	(footprint "Resistor_THT:R_Axial_DIN0204_L3.6mm_D1.6mm_P2.54mm_Vertical"
 		(layer "F.Cu")
-		(at 144.8 135.2 180)
+		(at 144.94 134 180)
 		(descr "Resistor, Axial_DIN0204 series, Axial, Vertical, pin pitch=2.54mm, 0.167W, length*diameter=3.6*1.6mm^2, http://cdn-reichelt.de/documents/datenblatt/B400/1_4W%23YAG.pdf")
 		(tags "Resistor Axial_DIN0204 series Axial Vertical pin pitch 2.54mm 0.167W length 3.6mm diameter 1.6mm")
@@
 	)
 	(segment
-		(start 155.8 109.2)
-		(end 157.8 111.2)
+		(start 149.745 109.2)
+		(end 155.8 109.2)
 		(width 0.5)
 		(layer "B.Cu")
@@
 	)
 	(segment
-		(start 144.83 114.115)
-		(end 149.745 109.2)
+		(start 157.8 111.2)
+		(end 166.38 111.2)
 		(width 0.5)
 		(layer "B.Cu")
@@
 	)
 	(segment
-		(start 157.8 111.2)
-		(end 166.38 111.2)
+		(start 155.8 109.2)
+		(end 157.8 111.2)
 		(width 0.5)
 		(layer "B.Cu")
@@
 	)
 	(segment
-		(start 149.745 109.2)
-		(end 155.8 109.2)
+		(start 144 114.94)
+		(end 144.005 114.94)
+		(width 0.5)
+		(layer "B.Cu")
+		(net 14)
+	)
+	(segment
+		(start 144.005 114.94)
+		(end 149.745 109.2)
 		(width 0.5)
 		(layer "B.Cu")
@@
 	)
 	(segment
-		(start 136 106.975)
-		(end 136.2 106.975)
+		(start 138.601627 109.376627)
+		(end 138.601627 112.525686)
 		(width 0.5)
 		(layer "F.Cu")
@@
 	(segment
 		(start 136.2 106.975)
-		(end 140.8 111.575)
+		(end 138.601627 109.376627)
+		(width 0.5)
+		(layer "F.Cu")
+		(net 17)
+	)
+	(segment
+		(start 136 106.975)
+		(end 136.2 106.975)
 		(width 0.5)
 		(layer "F.Cu")
@@
 	)
 	(segment
-		(start 152.08 135)
-		(end 152.08 139.2)
+		(start 152.06 139.22)
+		(end 152.02 139.26)
 		(width 0.5)
 		(layer "F.Cu")
@@
 	)
 	(segment
-		(start 142.4 135.34)
-		(end 142.26 135.2)
+		(start 152.06 134)
+		(end 152.06 139.22)
 		(width 0.5)
 		(layer "F.Cu")
-		(net 19)
+		(net 18)
 	)
 	(segment
-		(start 142.4 139.46)
-		(end 142.4 135.34)
+		(start 142.4 134)
+		(end 142.4 139.46)
 		(width 0.5)
 		(layer "F.Cu")
@@
 	)
 	(segment
-		(start 143.975 106.975)
-		(end 143.975 111.081)
+		(start 143.975 112.375)
+		(end 144 112.4)
 		(width 0.5)
 		(layer "F.Cu")
@@
 	)
 	(segment
-		(start 143.975 111.081)
-		(end 144.469 111.575)
+		(start 143.975 106.975)
+		(end 143.975 112.375)
 		(width 0.5)
 		(layer "F.Cu")
@@
 	)
 	(segment
-		(start 144.86 135.14)
-		(end 144.8 135.2)
+		(start 151.14 118.82)
+		(end 146.78 123.18)
 		(width 0.5)
-		(layer "F.Cu")
+		(layer "B.Cu")
 		(net 21)
 	)
 	(segment
-		(start 146.6 123.36)
-		(end 146.6 133.4)
+		(start 146.78 132.16)
+		(end 144.94 134)
 		(width 0.5)
 		(layer "B.Cu")
@@
 	)
 	(segment
-		(start 146.6 133.4)
-		(end 144.8 135.2)
+		(start 146.78 123.18)
+		(end 146.78 132.16)
 		(width 0.5)
 		(layer "B.Cu")
@@
 	)
 	(segment
-		(start 151.14 118.82)
-		(end 146.6 123.36)
+		(start 148.6 128)
+		(end 148.6 127)
 		(width 0.5)
 		(layer "B.Cu")
-		(net 21)
+		(net 22)
 	)
 	(segment
-		(start 148.6 128.98)
-		(end 154.62 135)
+		(start 154.6 134)
+		(end 148.6 128)
 		(width 0.5)
 		(layer "B.Cu")
@@
 	)
 	(segment
-		(start 151.14 121.36)
-		(end 148.6 123.9)
+		(start 148.6 123.9)
+		(end 148.6 127)
 		(width 0.5)
 		(layer "B.Cu")
@@
 	)
 	(segment
-		(start 148.6 123.9)
-		(end 148.6 128.98)
+		(start 151.14 121.36)
+		(end 148.6 123.9)
 		(width 0.5)
 		(layer "B.Cu")
